File: hardware/V1/capstone.brd (EAGLE design)
At the start: 68.7 x 51.3 mm, 30 parts, among them J1 61300311121, J2 61300311121, U1 BMP388, U2 LSM9DS1TR, U3 RFM95W-915S2

Commit message: new board
Parts:
- removed R1, R2: 10k, resistor:R0603
- added C5: 100n, rcl:C0603
- moved C4 0.89 mm to (58.4, 23.7)
- renumbered D1 to PWR_LED, D4 to FIX_LED
Connections:
- removed net BMP388_ADR: R2.1, U1.5
- removed net BMP388_CS: R1.1, U1.6
- net +3V3: now also C5.1, U1.6; no longer R1.2, R2.2
- net GND: now also C5.2, U1.5
Routing:
- net +3V3: track 211.5 -> 198.4 mm
- net BMP388_ADR: track 6.32 -> 0.00 mm
- net BMP388_CS: track 3.57 -> 0.00 mm
- net GND: track 167.8 -> 165.1 mm
- net GPS_TX: track 105.8 -> 103.3 mm
Other:
- board size 68.7 x 51.3 mm -> 68.6 x 51.3 mm
- board text added: "GND"
- board text added: "SERVO"
