File: hardware/V2/untitled.sch (EAGLE design)
At the start: 29 parts, among them J1 61300311121, J2 61300311121, U1 BMP388, U2 LSM9DS1TR, U3 RFM95W-915S2

Commit message: new board
Parts:
- removed ANT1: (no value), adafruit:PINHD-1X1
- removed C1, C4: 10 uF, resistor:C-USC0603
- removed C3: 0.1 uF, resistor:C-USC0603
- removed D1, D2, D3, D4: HSMH-C190, LED:HSMH-C190
- removed J1, J2: 61300311121, Headers:61300311121
- removed R10: 470, resistor:R-US_R0603
- removed R11, R12, R13: 100 Ohm, resistor:R-US_R0603
- removed R5, R6, R7, R8, R9: 10k, resistor:R-US_R0603
- removed U3: RFM95W-915S2, RFM95W-915S2:RFM95W-915S2
- added ANT, GND, VIN: (no value), wirepad:2,54/0,9
- added H1, H2, H3, H4: MOUNT-HOLE2.8, holes:MOUNT-HOLE2.8
- added LED1, LED2, LED3, LED4: (no value), led:LEDCHIPLED_1206
- added RC1, RC2, S1, S2: (no value), pinhead:PINHD-1X3
- added U5: RFM95W-915S2, RFM95W-915S2:RFM95W-915S2
- C2: value 100 nF -> 0.1u; device resistor:C-USC0603 -> rcl:C-USC1206
- R1, R2: value 10k -> 100; device resistor:R-US_R0603 -> rcl:R-US_M1206
- R3, R4: value 4.7k -> 100; device resistor:R-US_R0603 -> rcl:R-US_M1206
- U1: value BMP388 -> ADAFRUIT_MPL3115A2_BAROMETER; device BMP388:BMP388 -> AERO_Eagle_Library:ADAFRUIT_MPL3115A2_BAROMETER
- U2: value LSM9DS1TR -> ADAFRUIT_MTK3339_GPS; device LSM9DS1TR:LSM9DS1TR -> AERO_Eagle_Library:ADAFRUIT_MTK3339_GPS
- U4: value (none) -> SPARKFUN_MPU9250_IMU; device adafruit:GPS_FGPMMOPA6H -> AERO_Eagle_Library:SPARKFUN_MPU9250_IMU
Connections:
- removed net +3V3: C3.2, C4.1, D1.A, R1.2, R2.2, R3.2, R4.1, R5.2, R6.2, R7.2, R8.2, R9.2, U$1.3.3V, U1.VDD, U1.VDDIO, U2.VDD, U2.VDDIO, U3.3.3V, U4.VCC
- removed net ANT1: ANT1.1, U3.ANT
- removed net BMP388_ADR: R2.1, U1.SDO
- removed net BMP388_CS: R1.1, U1.CSB
- removed net BMP388_INT: U1.INT
- removed net GPS_1PPS: U4.1PPS
- removed net GPS_CS: U$1.10/TX2/PWM, U3.NSS
- removed net GPS_RESET: U3.RESET
- removed net LSM_CS_AG: R7.1, U2.CS_A/G
- removed net LSM_CS_M: R8.1, U2.CS_M
- removed net LSM_DEN_AG: R9.1, U2.DEN_A/G
- removed net LSM_INT1_AG: U2.INT1_A/G
- removed net LSM_INT2_AG: U2.INT2_A/G
- removed net LSM_INT_M: U2.INT_M
- removed net LSM_M_RDY: U2.DRDY_M
- removed net LSM_SDO_AG: R5.1, U2.SDO_A/G
- removed net LSM_SDO_M: R6.1, U2.SDO_M
- removed net N$2: C2.1, U2.C1
- removed net N$3: D4.C, R10.2
- removed net N$4: D4.A, U4.3D-FIX
- removed net N$5: D1.C, R11.1
- removed net N$6: D2.C, R12.1
- removed net N$7: D3.C, R13.1
- removed net VBACKUP: U4.VBACKUP
- new net 3.3V: C2.1, U$1.3.3V, U1.VIN, U2.3.3V, U2.VIN, U4.VDD, U5.3.3V
- new net EN: U$1.14/A0, U5.NSS
- new net GPS_FIX: U$1.4/CAN-RX-PWM, U2.FIX
- new net LED1: R1.1, U$1.8/TX3
- new net LED2: R2.1, U$1.7/RX3
- new net LED3: R3.1, U$1.6/PWM
- new net LED4: R4.1, U$1.5/PWM
- new net N$11: LED4.A, R4.2
- new net N$8: LED1.A, R1.2
- new net RECVR1: RC1.1, U$1.22/A8/T/PWM
- new net RECVR2: RC2.1, U$1.23/A9/T/PWM
- new net RESET: U$1.15/A1/T, U5.RESET
- net GND: now also GND.P, LED1.C, LED2.C, LED3.C, LED4.C, RC1.3, RC2.3, S1.3, S2.3, U1.GND, U4.AD0, U4.FSYNC, U4.GND, U5.DIO0, U5.DIO1, U5.DIO2, U5.DIO3, U5.DIO4, U5.DIO5, U5.GND; no longer C1.2, C3.1, C4.2, J1.1, J2.1, R10.1, R11.2, R12.2, R13.2, U1.VSS, U3.DIO0, U3.DIO1, U3.DIO2, U3.DIO3, U3.DIO4, U3.DIO5, U3.GND, U4.GND@1, U4.GND@2, U4.GND@3, U4.GND@4
- net GPS_RX: now also U$1.10/TX2/PWM, U2.RX; no longer U4.RX
- net GPS_TX: now also U$1.9/RX2/PWM, U2.TX; no longer U4.TX
- net MISO: now also U5.MISO; no longer U3.MISO
- net MOSI: now also U5.MOSI; no longer U3.MOSI
- net N$1: now also ANT.P, U5.ANT; no longer C1.1, U2.CAP
- net N$10: now also LED3.A, R3.2; no longer D3.A
- net N$9: now also LED2.A, R2.2; no longer D2.A
- net SCK: now also U5.SCK; no longer U3.SCK
- net SCL: now also U1.SCL, U4.SCL; no longer R4.2, U1.SCK, U2.SCL/SPC
- net SDA: now also U1.SDA, U4.SDA; no longer R3.1, U1.SDI, U2.SDA/SDI/SDO
- net SERVO1: now also S1.1, U$1.20/A6/PWM; no longer J1.3, U$1.22/A8/T/PWM
- net SERVO2: now also S2.1, U$1.21/A7/PWM; no longer J2.3, U$1.23/A9/T/PWM
- net VIN: now also S1.2, S2.2, VIN.P; no longer J1.2, J2.2
Other:
- note removed: "3.3V Logic"
- note removed: "AG Data Enable"
- note removed: "BMP-388"
- note removed: "Ceramic Capacitor"
- note removed: "Could put a pull up and diode on RX to ensure 3.3V but Teensy3.2 is 3.3V"
- note removed: "Debug LEDs"
- note removed: "I2C Address is 111011x If SDO low, 1110110 (0x76) If SDO high, 1110111 (0x77)"
- note removed: "If CS pins are pulled high, use I2C mode"
- note removed: "No fix, LED pulse up and down every second Fix, LED pulse every 15 seconds"
- note removed: "Pull CS and SDO high when using I2C"
- note removed: "Pulse per second, used for uC syncing"
- note removed: "SDO_A/G LSB for A/G I2C Address Pulled high - 0x1E"
- note removed: "SDO_M LSB for Mag I2C Address Pulled high - 0x6B"
- note removed: "Servo Headers"
- note removed: "VSS is GND"
