File: hardware/V5 - Prototype Design/capstone.brd (EAGLE design)
At the start: 74 x 61.8 mm, 25 parts, among them U1 ADAFRUIT_MPL3115A2_BAROMETER, U2 ADAFRUIT_MTK3339_GPS, U4 SPARKFUN_MPU9250_IMU, U5 RFM95W-915S2

Commit message: Schematic Cleanup
Routing:
- net SERVO3: track 19.1 -> 14.0 mm
- net GPS_FIX: track 54.6 -> 50.8 mm
- net LED1: track 57.1 -> 55.9 mm
Changed lines of the file:
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@@
 <contactref element="U4" pad="AD0"/>
 <contactref element="RC3" pad="3"/>
+<contactref element="J1" pad="1"/>
 <contactref element="S3" pad="3"/>
-<contactref element="J1" pad="1"/>
+<wire x1="56.106" y1="57.15" x2="61.948" y2="57.15" width="0" layer="19" extent="1-1"/>
+<wire x1="50.8" y1="59.69" x2="56.106" y2="59.662" width="0" layer="19" extent="1-1"/>
+<wire x1="41.99" y1="56.53" x2="50.391" y2="57.15" width="0" layer="19" extent="1-1"/>
+<wire x1="41.99" y1="48.53" x2="41.99" y2="54.53" width="0" layer="19" extent="1-1"/>
+<wire x1="33.02" y1="57.15" x2="39.243" y2="56.515" width="0" layer="19" extent="1-1"/>
+<wire x1="34.29" y1="35.56" x2="39.243" y2="44.45" width="0" layer="19" extent="1-1"/>
+<wire x1="29.21" y1="42.545" x2="34.29" y2="35.56" width="0" layer="19" extent="1-1"/>
+<wire x1="16.383" y1="57.785" x2="26.59" y2="56.53" width="0" layer="19" extent="1-1"/>
+<wire x1="15.748" y1="48.26" x2="16.383" y2="57.785" width="0" layer="19" extent="1-1"/>
+<wire x1="10.668" y1="40.64" x2="15.748" y2="48.26" width="0" layer="19" extent="1-1"/>
+<wire x1="10.668" y1="33.02" x2="10.668" y2="40.64" width="0" layer="19" extent="1-1"/>
+<wire x1="54.61" y1="44.45" x2="41.99" y2="44.53" width="0" layer="19" extent="1-1"/>
+<wire x1="17.78" y1="14.605" x2="10.668" y2="33.02" width="0" layer="19" extent="1-1"/>
+<wire x1="16.51" y1="2.54" x2="17.78" y2="14.605" width="0" layer="19" extent="1-1"/>
+<wire x1="20.32" y1="2.54" x2="16.51" y2="2.54" width="0" layer="19" extent="1-1"/>
+<wire x1="12.7" y1="2.54" x2="16.51" y2="2.54" width="0" layer="19" extent="1-1"/>
+<wire x1="41.91" y1="2.54" x2="20.32" y2="2.54" width="0" layer="19" extent="1-1"/>
+<wire x1="48.26" y1="2.54" x2="41.91" y2="2.54" width="0" layer="19" extent="1-1"/>
+<wire x1="52.07" y1="2.54" x2="48.26" y2="2.54" width="0" layer="19" extent="1-1"/>
+<wire x1="55.88" y1="2.54" x2="52.07" y2="2.54" width="0" layer="19" extent="1-1"/>
+<wire x1="63.5" y1="5.08" x2="55.88" y2="2.54" width="0" layer="19" extent="1-1"/>
 </signal>
 <signal name="AGND">
@@
 <contactref element="U5" pad="13"/>
 <contactref element="U2" pad="3.3V"/>
-<contactref element="U2" pad="VIN"/>
 <contactref element="U4" pad="VDD"/>
 <wire x1="41.99" y1="50.53" x2="39.259" y2="50.53" width="0.1524" layer="1"/>
@@
 <contactref element="U$1" pad="3.3V"/>
 <contactref element="U$1" pad="3.3V1"/>
+<contactref element="U2" pad="VIN"/>
+<wire x1="52.07" y1="44.45" x2="69.85" y2="44.45" width="0" layer="19" extent="1-1"/>
+<wire x1="41.99" y1="50.53" x2="52.07" y2="44.45" width="0" layer="19" extent="1-1"/>
+<wire x1="35.69" y1="59.309" x2="39.243" y2="50.546" width="0" layer="19" extent="1-1"/>
+<wire x1="36.83" y1="35.56" x2="39.259" y2="50.53" width="0" layer="19" extent="1-1"/>
+<wire x1="13.208" y1="33.02" x2="36.83" y2="35.56" width="0" layer="19" extent="1-1"/>
+<wire x1="17.78" y1="12.065" x2="13.208" y2="33.02" width="0" layer="19" extent="1-1"/>
+<wire x1="26.67" y1="7.62" x2="17.78" y2="12.065" width="0" layer="19" extent="1-1"/>
 </signal>
 <signal name="VBAT">
@@
 <signal name="LED1">
 <contactref element="R1" pad="1"/>
-<contactref element="U$1" pad="8"/>
 <wire x1="14.1" y1="54.737" x2="21.336" y2="54.737" width="0.1524" layer="1"/>
 <via x="21.336" y="54.737" extent="1-16" drill="0.35"/>
@@
 <via x="40.64" y="40.64" extent="1-16" drill="0.35"/>
 <wire x1="40.64" y1="40.64" x2="40.64" y2="25.4" width="0.1524" layer="16"/>
-<wire x1="40.64" y1="25.4" x2="41.91" y2="25.4" width="0.1524" layer="16"/>
+<contactref element="U$1" pad="8"/>
+<wire x1="40.64" y1="25.4" x2="41.91" y2="25.4" width="0" layer="19" extent="16-16"/>
 </signal>
 <signal name="LED2">
@@
 <wire x1="62.23" y1="25.4" x2="45.72" y2="25.4" width="0.1524" layer="1"/>
 <via x="45.72" y="25.4" extent="1-16" drill="0.35"/>
-<contactref element="U$1" pad="2"/>
-<wire x1="41.91" y1="10.16" x2="45.72" y2="10.16" width="0.1524" layer="1"/>
 <via x="45.72" y="10.16" extent="1-16" drill="0.35"/>
 <wire x1="45.72" y1="25.4" x2="45.72" y2="10.16" width="0.1524" layer="16"/>
+<contactref element="U$1" pad="2"/>
+<wire x1="41.91" y1="10.16" x2="45.72" y2="10.16" width="0" layer="19" extent="1-1"/>
 </signal>
 <signal name="RADIO_INT">
@@
 <signal name="SERVO3">
 <contactref element="U$1" pad="3"/>
+<wire x1="41.91" y1="12.7" x2="55.88" y2="12.7" width="0.1524" layer="1"/>
+<via x="55.88" y="12.7" extent="1-16" drill="0.35"/>
 <contactref element="S3" pad="1"/>
-<wire x1="41.91" y1="12.7" x2="55.88" y2="12.7" width="0.1524" layer="1"/>
-<wire x1="55.88" y1="7.62" x2="55.88" y2="12.7" width="0.1524" layer="16"/>
-<via x="55.88" y="12.7" extent="1-16" drill="0.35"/>
+<wire x1="55.88" y1="12.7" x2="55.88" y2="7.62" width="0" layer="19" extent="1-1"/>
 </signal>
 <signal name="RECVR3">
